File: hard/carte_mere_mbed/carte_mere_mbed.sch (EAGLE design)
At the start: 0 parts

Commit message: Début carte mère
Début du schématic de la carte mère
Parts:
- added C10: 330nF, rcl:C-EUC0805
- added C11: 2200u, rcl:CPOL-EUTT5D11
- added C9: 100nF, rcl:C-EUC0805
- added CAN: Micromatch 8p, jt-con-micromatch:MMATCH-8-PTH
- added F2: (no value), fuse:SHK20Q
- added IC2: 7805TV, linear:7805TV
- added JP1, JP5: AX12, SparkFun-Connectors:M03POLAR
- added LED_12V_DIRTY, LED_5V_DIRTY, LED_5V_µP: (no value), adafruit:LEDCHIPLED_0805
- added NUCLEO1: MBED-NUCLEO-F401RE-MORPHO, mbed-nucleo:MBED-NUCLEO-F401RE-MORPHONUCLEOF401RE-MORPHO
- added R1, R6: 400, SparkFun-Passives:RESISTOR0805-RES
- added R2: 4,7k, rcl:R-EU_M0805
- added R5: 10k, rcl:R-EU_M0805
- added R7: 1k, SparkFun-Passives:RESISTOR0805-RES
- added SHARP1, SHARP2, SHARP3, SHARP4, SHARP5, SHARP6: (no value), con-lstb:MA03-1
- added U1: MCP2551, SparkFun-DigitalIC:MCP2551
- added U2: ADUM1250ARZ, Analog Devices_By_element14_Batch_1:ADUM1250ARZ
- added X2: 5V, con-weidmueller-sl35:90-2
- added X3: 12V Dirty, con-weidmueller-sl35:90-2
Connections:
- new net +12V: C11.+, JP1.2, JP5.2, R5.2, R7.1, X3.1
- new net +5V: C9.2, IC2.VO, R6.1, U2.VDD2
- new net CANH: CAN.4, CAN.5, U1.CANH
- new net CANL: CAN.3, CAN.6, U1.CANL
- new net GND1: CAN.1, CAN.8, LED_5V_µP.C, NUCLEO1.GND/SERIAL1_RX, NUCLEO1.GND_0, NUCLEO1.GND_1, NUCLEO1.GND_2, NUCLEO1.GND_3, NUCLEO1.GND_4, R2.1, SHARP1.3, SHARP2.3, SHARP3.3, SHARP4.3, SHARP5.3, SHARP6.3, U1.VSS, U2.GND1, X2.2
- new net GND2: C10.1, C11.-, C9.1, F2.1A, IC2.GND, JP1.1, JP5.1, LED_12V_DIRTY.C, LED_5V_DIRTY.C, U2.GND2
- new net N$11: LED_12V_DIRTY.A, R7.2
- new net N$12: LED_5V_µP.A, R1.2
- new net N$2: LED_5V_DIRTY.A, R6.2
- new net N$27: F2.2A, X3.2
- new net N$3: U1.RXD
- new net N$32: C10.2, IC2.VI
- new net N$4: R2.2, U1.RS
- new net N$5: U1.TXD
- new net SHARP0: NUCLEO1.PA_0/A_IN/A0/PWM2-1, SHARP1.2
- new net SHARP1: NUCLEO1.PA_1/A_IN/A1/PWM2-2, SHARP2.2
- new net SHARP2: NUCLEO1.PA_4/A_IN/A2/SPI1_NSS, SHARP3.2
- new net SHARP3: NUCLEO1.PB_0/A_IN/A3/PWM1-2N, SHARP4.2
- new net SHARP4: NUCLEO1.PC_1/A_IN/A4, SHARP5.2
- new net SHARP5: NUCLEO1.PC_0/A_IN/A5, SHARP6.2
- new net UART6_CLEAN: NUCLEO1.PA_11/PWM1-4/SERIAL6_TX, NUCLEO1.PA_12/SERIAL6_RX, U2.SCL1
- new net UART6_DIRTY: JP1.3, JP5.3, R5.1, U2.SCL2
- new net VCC: CAN.2, CAN.7, NUCLEO1.VIN(5V-9V), R1.1, SHARP1.1, SHARP2.1, SHARP3.1, SHARP4.1, SHARP5.1, SHARP6.1, U1.VDD, U2.VDD1, X2.1
Other:
- note added: "Alimentation CLEAN"
- note added: "Alimentation DIRTY"
- note added: "CLEAN"
- note added: "Carte Nucleo"
- note added: "Connexion CAN"
- note added: "Connexions AX12"
- note added: "Connexions Sharp"
- note added: "DIRTY"
