File: hard/carte_mere_mbed/carte_mere_mbed.sch (EAGLE design)
At the start: 27 parts, among them IC2 7805TV, U1 MCP2551, U2 ADUM1250ARZ, X2 5V, X3 12V Dirty

Commit message: Avancé de la carte mere
Parts:
- added C1, C2: 22u, SparkFun-Capacitors:CAP_POLPTH1
- added I2C: Micromatch 8p, jt-con-micromatch:MMATCH-8-PTH
- added LED1: (no value), adafruit:LEDCHIPLED_0805
- added ODO0, ODO1, ODO2, US1, US2, US3, US4, US5: (no value), con-lstb:MA04-1
- added R3: (no value), SparkFun-Resistors:RESISTOR0805-RES
Connections:
- new net CHA0: ODO0.2
- new net CHA1: ODO1.2
- new net CHA2: ODO2.2
- new net CHB0: ODO0.3
- new net CHB1: ODO1.3
- new net CHB2: ODO2.3
- new net ECHO0: NUCLEO1.PA_13, US1.3
- new net ECHO1: NUCLEO1.PA_15/PWM2-1/SPI1_NSS, US2.3
- new net ECHO2: NUCLEO1.PC_13/USER_BUTTON, US3.3
- new net ECHO3: NUCLEO1.PC_15, US4.3
- new net ECHO4: NUCLEO1.PH_1, US5.3
- new net N$1: NUCLEO1.PC_10/SPI3_SCK, R3.2
- new net N$6: LED1.A, R3.1
- new net SCL: I2C.4, I2C.5, NUCLEO1.PB_8/D15/PWM4-3/I2C1-SCL
- new net SDA: I2C.2, I2C.7, NUCLEO1.PB_9/D14/PWM4-4/I2C1-SDA/SPI2_NSS
- new net TRIG0: NUCLEO1.PC_12/SPI3_MOSI, US1.2
- new net TRIG1: NUCLEO1.PA_14, US2.2
- new net TRIG2: NUCLEO1.PB_7/PWM4-2/I2C1_SDA, US3.2
- new net TRIG3: NUCLEO1.PC_14, US4.2
- new net TRIG4: NUCLEO1.PH_0, US5.2
- net GND1: now also C1.-, C2.-, I2C.1, I2C.8, LED1.C, ODO0.4, ODO1.4, ODO2.4, SHARP1.2, SHARP2.2, SHARP3.2, SHARP4.2, SHARP5.2, SHARP6.2, US1.1, US2.1, US3.1, US4.1, US5.1; no longer SHARP1.3, SHARP2.3, SHARP3.3, SHARP4.3, SHARP5.3, SHARP6.3
- net SHARP0: now also NUCLEO1.PC_5/A_IN, SHARP1.1; no longer NUCLEO1.PA_0/A_IN/A0/PWM2-1, SHARP1.2
- net SHARP1: now also NUCLEO1.PB_1/A_IN/PWM1-3N, SHARP2.1; no longer NUCLEO1.PA_1/A_IN/A1/PWM2-2, SHARP2.2
- net SHARP2: now also NUCLEO1.PC_4/A_IN, SHARP3.1; no longer NUCLEO1.PA_4/A_IN/A2/SPI1_NSS, SHARP3.2
- net SHARP3: now also NUCLEO1.PC_3/A_IN/SPI2-MOSI, SHARP4.1; no longer NUCLEO1.PB_0/A_IN/A3/PWM1-2N, SHARP4.2
- net SHARP4: now also NUCLEO1.PC_2/A_IN/SPI2_MISO, SHARP5.1; no longer NUCLEO1.PC_1/A_IN/A4, SHARP5.2
- net SHARP5: now also SHARP6.1; no longer SHARP6.2
- net VCC: now also C1.+, C2.+, I2C.3, I2C.6, ODO0.1, ODO1.1, ODO2.1, SHARP1.3, SHARP2.3, SHARP3.3, SHARP4.3, SHARP5.3, SHARP6.3, US1.4, US2.4, US3.4, US4.4, US5.4; no longer SHARP1.1, SHARP2.1, SHARP3.1, SHARP4.1, SHARP5.1, SHARP6.1
Other:
- note added: "Connexion I2C"
- note added: "Connexions US"
- note added: "Odometri"
- moved on the sheet: LED_5V_µP, R1, X2
