File: hard/carte_moteur/cartev0/ares2015_motor_v0.sch (EAGLE design)
At the start: 60 parts, among them CN1 1X4-CLEANBIG, IC1 TB6612FNG, J1 1X5, Q1 AOD417, U1 DRV8828PWP, U2 PCA9685

Commit message: maj schema carte moteur (80% de schema finit)
Parts:
- removed C10, C6: 10uF, adafruit:C-USC0805K
- removed C12: 330nF, rcl:C-EUC0805
- removed C13: 2200u, rcl:CPOL-EUTT5D11
- removed C9: 100uF, adafruit:CPOL-USC
- removed CN1: 1X4-CLEANBIG, adafruit:1X4-CLEANBIG
- removed D0-7, JP2: (no value), adafruit:PINHD-1X8CLEANBIG
- removed IN: SL-3.5-2-90G, WEIDMULLER:SL-3.5-2-90G
- removed J1: 1X5, adafruit:1X5
- removed JP1: (no value), microbuilder:HEADER-1X476MIL
- removed JP3: (no value), microbuilder:HEADER-1X1070MIL
- removed MPOWER, SERPWR: 1X2-3.5MM, adafruit:1X2-3.5MM
- removed R7, R8: 10K, adafruit:R-US_R0805
- removed SERVO1, SERVO2: (no value), adafruit:PINHD-1X3
- removed SJ1: (no value), microbuilder:SOLDERJUMPER_2WAY
- removed U$6: L7805TO263, st-microelectronics:L7805TO263
- added C14: 0.1uF, adafruit:C-USC0805K
- added IC2: (no value), SparkFun-PowerIC:V_REG_LM1117SOT223
- added IN_MOT1, OUT_MOT1: SL-3.5-2-90G, WEIDMULLER:SL-3.5-2-90G
- added PWR1: (no value), jumper:JP1E
- added R11: 135k, adafruit:R-US_R0805
- added R12, R13, R14: 1.5k, adafruit:R-US_R0805
- C1: value 0.1uF -> 0.47uF
- C11: value 100nF -> 0.1uF; device rcl:C-EUC0805 -> adafruit:C-USC0805K
- IC1: value TB6612FNG -> ISO7220A; device adafruit:TB6612FNG -> texas:ISO7220A
Connections:
- removed net +3V3: JP2.5, SJ1.3, U$1.3V, U$5.3V
- removed net +5V: C11.2, C9.+, JP2.4, SERPWR.1, SERVO1.2, SERVO2.2, SJ1.1, U$1.5V, U$5.5V, U$6.OUT
- removed net GNDA: C11.1, C12.1, C13.-, IN.1, U$6.GND
- removed net N$16: U1.OUT1_2
- removed net N$33: U1.OUT2
- removed net N$7: IC1.BO2, IC1.BO2', J1.2
- removed net PWM1A: JP3.9, SERVO2.3, U$1.D9, U$5.D9
- new net GND_CLEAN: C2.2, IC1.GND2, PWR1.2, U$1.GND@1, U$1.GND@2, U$5.GND@1, U$5.GND@2
- new net N$12: OUT_MOT1.2, U1.OUT2, U1.OUT2_2
- new net N$14: OUT_MOT1.1, U1.OUT1, U1.OUT1_2
- new net N$15: U$1.A5/SCL, U$5.A5/SCL
- new net N$17: U$1.A4/SDA, U$5.A4/SDA
- new net N$34: U$1.GND, U$5.GND
- new net SCL_CLEAN: IC1.OUTB, R11.1, U$1.SCL, U$5.SCL
- new net SDA_CLEAN: IC1.OUTA, R12.1, U$1.SDA, U$5.SDA
- new net VCC_CLEAN: C2.1, IC1.VCC2, R11.2, R12.2, U$1.3V, U$5.3V
- net +12V: now also IC2.IN; no longer C12.2, C13.+, IC1.VM1, IC1.VM2, IC1.VM3, IN.2, U$6.IN
- net /RST: no longer JP2.6
- net GND: now also C11.2, C14.2, IC1.GND1, IC2.ADJ, IN_MOT1.1, PWR1.1; no longer C10.2, C2.2, C6.2, C9.-, IC1.GND, IC1.PGND1, IC1.PGND1', IC1.PGND2, IC1.PGND2', J1.3, JP2.2, JP2.3, JP3.4, MPOWER.1, SERPWR.2, SERVO1.1, SERVO2.1, U$1.GND, U$1.GND@1, U$1.GND@2, U$5.GND, U$5.GND@1, U$5.GND@2
- net N$1: no longer JP2.7
- net N$140: now also IN_MOT1.2; no longer MPOWER.2
- net N$18: now also IC1.INA, R13.1; no longer U1.OUT2_2
- net N$19: now also IC1.INB, R14.1; no longer U1.OUT1
- net N$2: no longer JP2.8
- net N$20: no longer CN1.4
- net N$21: no longer CN1.3
- net N$22: no longer CN1.2
- net N$23: no longer CN1.1
- net N$24: no longer D0-7.1
- net N$25: no longer D0-7.2
- net N$26: no longer D0-7.3
- net N$27: no longer D0-7.5
- net N$28: no longer D0-7.8
- net N$29: no longer JP3.10
- net N$30: no longer JP3.6
- net N$31: no longer JP3.5
- net N$32: no longer JP3.3
- net N$4: now also U$1.D9, U$5.D9; no longer IC1.AO1, IC1.AO1', J1.5
- net N$6: now also U1.ENBL; no longer IC1.AO2, IC1.AO2', J1.4
- net N$9: now also U$1.5V, U$5.5V; no longer IC1.BO1, IC1.BO1', J1.1
- net PWM0: no longer JP1.1
- net PWM0A: no longer D0-7.7
- net PWM0B: no longer D0-7.6
- net PWM1: no longer JP1.2
- net PWM10: no longer IC1.AIN1
- net PWM11: no longer IC1.BIN1
- net PWM12: no longer IC1.BIN2
- net PWM13: no longer IC1.PWMB
- net PWM14: no longer JP1.3
- net PWM15: no longer JP1.4
- net PWM1B: no longer JP3.8, SERVO1.3
- net PWM2A: no longer JP3.7
- net PWM2B: no longer D0-7.4
- net PWM8: no longer IC1.PWMA
- net PWM9: no longer IC1.AIN2
- net SCL: no longer JP3.1, R8.1, U$1.A5/SCL, U$1.SCL, U$5.A5/SCL, U$5.SCL
- net SDA: no longer JP3.2, R7.1, U$1.A4/SDA, U$1.SDA, U$5.A4/SDA, U$5.SDA
- net V3POUT1: now also C1.1
- net VCC: now also C11.1, C14.1, IC1.VCC1, IC2.OUT, IC2.OUT@1; no longer C1.1, C10.1, C2.1, C6.1, IC1.STBY, IC1.VCC, R7.2, R8.2, SJ1.2
- net VIN: no longer JP2.1
Other:
- note added: "Générateur PWM"
- note added: "ISO1541 (isolateur bus I2C)"
- note added: "Permet de choisir par des soudure 5 bits sur l'identifiant de l'I2C"
- note added: "Permet de relier le GND_CLEAN au GND et 12V à VIN (et eviter l'utilisation de la carte alim)"
- moved on the sheet: A0, A1, A2, A3, A4, C1, C11, C2, C3, C4, C5, C8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
