File: hard/carte_moteur/carte_moteur_v0/ares2015_motor_v0.brd (EAGLE design)
At the start: 68.6 x 53.3 mm, 50 parts, among them IC1 ISO7220A, Q1 AOD417, U1 DRV8828PWP, U2 PCA9685

Commit message: schematic de la carte moteur finit !
Parts:
- removed A2, A3, A4: (no value), jumper:SJ
- removed HEADER: (no value), con-lsta:FE06
- removed TP1, TP2, TP3: (no value), microbuilder:TESTPOINT_ROUND_2MM
- added C10, C15, C18: 0.47uF, adafruit:C0805K
- added C12, C16, C6: 0.01uF, adafruit:C0805K
- added C13, C17, C3, C9: 0.1uF, adafruit:C0805K
- added LED3, LED4, LED5: rouge, adafruit:CHIPLED_0805
- added MOTOR1, MOTOR2, MOTOR3: DRV8828PWP, Texas Instruments_By_element14_Batch_1:SOP65P640X120-29N
- added OUT_MOT0, OUT_MOT2, OUT_MOT3: SL-3.5-2-90G, WEIDMULLER:SL-3.5-2-90G
- added PWM_ACCES1: MMATCH-6-, jt-con-micromatch:AMP-215079-6
- added R15: 0.25, adafruit:R0805
- added U$6: LMD128D818, ADS128D818:ADC128D818
- R3, R6: value 10k -> 330
- R5: value 10k -> 0.25
- R7: value 10K -> 0.25
- R8: value 10K -> 330
- moved R8 277.6 mm to (-39.6, -224.4), turned to 0 degrees
- moved R7 235.6 mm to (-20.4, -185.0), turned to 0 degrees
- moved R6 219.5 mm to (-39.6, -193.5), turned to 0 degrees
- moved R3 192.3 mm to (-39.6, -162.7), turned to 0 degrees
- moved R5 177.0 mm to (-20.4, -154.2), turned to 0 degrees
- moved OUT_MOT1 131.5 mm to (-31.1, -155.7)
- renumbered IC2 to 3V3LDO, INPUT to PWM_ACCES, U1 to MOTOR0
Connections:
- net VIN renamed VIN_ARDUINO
- removed net C_DIR1: HEADER.4, PWM_ACCES.3
- removed net C_DIR2: HEADER.2, PWM_ACCES.5
- removed net C_PWM1: HEADER.3, PWM_ACCES.4
- removed net C_PWM2: HEADER.1, PWM_ACCES.6
- new net ADC0: MOTOR0.6, MOTOR0.9, R10.1, U$6.16
- new net ADC1: MOTOR1.6, MOTOR1.9, R5.1, U$6.15
- new net ADC2: MOTOR2.6, MOTOR2.9, R7.1, U$6.14
- new net ADC3: MOTOR3.6, MOTOR3.9, R15.1, U$6.13
- new net ADC4: U$6.12
- new net ADC5: U$6.11
- new net ADC6: U$6.10
- new net ADC7: U$6.9
- new net N$16: MOTOR0.10, MOTOR0.5, OUT_MOT0.1
- new net N$33: MOTOR1.10, MOTOR1.5, OUT_MOT1.1
- new net N$38: C12.1, MOTOR2.1
- new net N$40: C12.2, MOTOR2.2
- new net N$41: C13.1, MOTOR2.3
- new net N$42: LED4.C, MOTOR2.18
- new net N$43: LED4.A, R6.2
- new net N$46: MOTOR2.10, MOTOR2.5, OUT_MOT2.1
- new net N$47: MOTOR2.7, MOTOR2.8, OUT_MOT2.2
- new net N$48: C16.1, MOTOR3.1
- new net N$50: C17.1, MOTOR3.3
- new net N$51: LED5.C, MOTOR3.18
- new net N$52: LED5.A, R8.2
- new net N$53: MOTOR3.10, MOTOR3.5, OUT_MOT3.1
- new net N$54: MOTOR3.7, MOTOR3.8, OUT_MOT3.2
- new net V3POUT0: C1.1, MOTOR0.12, MOTOR0.13, MOTOR0.15
- new net V3POUT2: C15.1, MOTOR2.12, MOTOR2.13, MOTOR2.15
- new net V3POUT3: C18.1, MOTOR3.12, MOTOR3.13, MOTOR3.15
- net +12V: now also C13.2, C17.2, C9.2, MOTOR1.11, MOTOR1.4, MOTOR2.11, MOTOR2.4, MOTOR3.11, MOTOR3.4
- net A0: now also U$6.7
- net A1: now also U$6.8
- net A2: no longer A2.2, R3.2, TP3.P$1
- net A3: no longer A3.1, R5.2, TP2.P$1
- net A4: no longer A4.1, R6.2, TP1.P$1
- net GND: now also C10.2, C15.2, C18.2, C3.2, MOTOR1.14, MOTOR1.28, MOTOR1.29, MOTOR2.14, MOTOR2.28, MOTOR2.29, MOTOR3.14, MOTOR3.28, MOTOR3.29, PWM_ACCES1.2, R15.2, R5.2, R7.2, U$6.4; no longer HEADER.5, R3.1, R5.1, R6.1
- net N$12: now also C6.2, MOTOR1.2; no longer MOTOR0.7, MOTOR0.8, OUT_MOT1.2
- net N$14: now also C9.1, MOTOR1.3; no longer MOTOR0.10, MOTOR0.5, OUT_MOT1.1
- net N$18: now also LED3.C, MOTOR1.18; no longer IC1.2, R13.1
- net N$19: now also LED3.A, R3.2; no longer IC1.3, R14.1
- net N$35: now also MOTOR1.7, MOTOR1.8, OUT_MOT1.2; no longer MOTOR0.6, MOTOR0.9, R10.1
- net N$49: now also C16.2, MOTOR3.2; no longer MOTOR0.20
- net N$6: now also C6.1, MOTOR1.1; no longer MOTOR0.21
- net N$7: now also MOTOR0.7, MOTOR0.8, OUT_MOT0.2; no longer IC1.1
- net PWM0: now also MOTOR0.21, PWM_ACCES.4
- net PWM1: now also MOTOR0.20, PWM_ACCES.3
- net PWM2: now also MOTOR1.21, PWM_ACCES.6
- net PWM3: now also MOTOR1.20, PWM_ACCES.5
- net PWM4: now also MOTOR2.21, PWM_ACCES1.4
- net PWM5: now also MOTOR2.20, PWM_ACCES1.3
- net PWM6: now also MOTOR3.21, PWM_ACCES1.6
- net PWM7: now also MOTOR3.20, PWM_ACCES1.5
- net SCL: now also IC1.3, R14.1, U$6.3; no longer R8.1, U$1.SCL, U$5.SCL
- net SCL_CLEAN: now also U$1.SCL, U$5.SCL
- net SDA: now also IC1.2, R13.1, U$6.2; no longer R7.1, U$1.SDA, U$5.SDA
- net SDA_CLEAN: now also U$1.SDA, U$5.SDA
- net V3POUT1: now also C10.1, MOTOR1.12, MOTOR1.13, MOTOR1.15; no longer C1.1, MOTOR0.12, MOTOR0.13, MOTOR0.15
- net VCC: now also C3.1, IC1.1, MOTOR1.16, MOTOR1.17, MOTOR1.19, MOTOR1.23, MOTOR1.24, MOTOR1.25, MOTOR1.26, MOTOR1.27, MOTOR2.16, MOTOR2.17, MOTOR2.19, MOTOR2.23, MOTOR2.24, MOTOR2.25, MOTOR2.26, MOTOR2.27, MOTOR3.16, MOTOR3.17, MOTOR3.19, MOTOR3.23, MOTOR3.24, MOTOR3.25, MOTOR3.26, MOTOR3.27, PWM_ACCES1.1, R13.2, R14.2, R3.1, R6.1, R8.1, U$6.5; no longer A2.1, A3.2, A4.2, HEADER.6, R7.2, R8.2
Routing:
- net VCC: track 11.7 -> 3.81 mm
- net A3: track 24.5 -> 17.4 mm, vias 1 -> 0
- net A2: track 14.3 -> 7.44 mm, vias 1 -> 0
- net A4: track 23.4 -> 17.0 mm, vias 1 -> 0

Commit message: modifs mineures
Parts:
- removed U$2, U$3, U$4: FIDUCIAL, adafruit:FIDUCIAL_1MM
- IC1: value ISO7220A -> ISO1541
- R1, R10, R12, R13, R14, R15, R2, R3, R4, R5, R6, R7, R8, R9: device adafruit:R0805 -> adafruit:M0805
- R11: value 135k -> 1.5k; device adafruit:R0805 -> adafruit:M0805
- moved C3 173.5 mm to (25.8, 31.0)
- moved C2 169.7 mm to (25.3, 43.1), turned to 270 degrees
- moved R14 168.6 mm to (19.4, 33.1), turned to 180 degrees
- moved R12 165.2 mm to (20.4, 45.1)
- moved R13 162.8 mm to (14.9, 34.0), turned to 90 degrees
- moved R11 161.7 mm to (19.2, 47.4), turned to 180 degrees
- moved IC1 146.9 mm to (20.1, 39.1)
- moved C1 137.4 mm to (30.7, 34.2), turned to 270 degrees
- moved C11 124.7 mm to (29.2, 25.5), turned to 270 degrees
- moved PWR1 122.7 mm to (42.9, 7.24), turned to 180 degrees
- moved C14 112.4 mm to (12.8, 23.9), turned to 270 degrees
- moved 3V3LDO 104.4 mm to (5.59, 24.9), turned to 90 degrees
- moved OUT_MOT0 95.9 mm to (55.4, 43.6), turned to 180 degrees
- moved R10 86.6 mm to (50.2, 42.2)
- moved R9 80.6 mm to (43.4, 46.6)
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Routing:
- net +12V: track 78.5 -> 22.0 mm
- net SCL: track 51.7 -> 0.00 mm, vias 1 -> 0
- net VIN_ARDUINO: track 26.2 -> 0.00 mm
- net A3: track 17.4 -> 0.00 mm
- net A4: track 17.0 -> 0.00 mm
- net A2: track 7.44 -> 0.00 mm

Commit message: routage : automatique=98,8% réussite. Reste à ajouter les deux autres hacheurs
Parts:
- removed C12, C16: 0.01uF, adafruit:C0805K
- removed C13, C17: 0.1uF, adafruit:C0805K
- removed C15, C18: 0.47uF, adafruit:C0805K
- removed LED4, LED5: rouge, adafruit:CHIPLED_0805
- removed MOTOR2, MOTOR3: DRV8828PWP, Texas Instruments_By_element14_Batch_1:SOP65P640X120-29N
- removed OUT_MOT2, OUT_MOT3: SL-3.5-2-90G, WEIDMULLER:SL-3.5-2-90G
- removed PWM_ACCES, PWM_ACCES1: MMATCH-6-, jt-con-micromatch:AMP-215079-6
- removed PWR, PWR1: (no value), jumper:JP1
- removed R15, R7: 0.25, adafruit:M0805
- removed R6, R8: 330, adafruit:M0805
- removed TP4, TP5: (no value), microbuilder:TESTPOINT_ROUND_2MM
- removed U$1, U$5: ARDUINO_R3_ICSP, adafruit:ARDUINOR3_ICSP
- added ALIM_GND, ALIM_V+: (no value), jumper:JP1
- added U1: ARDUINOR3-BPLACE, adafruit:ARDUINOR3-BPLACE
- moved C10 226.4 mm to (55.4, 48.0)
- moved R3 224.7 mm to (45.1, 45.5), turned to 180 degrees
- moved OUT_MOT1 219.8 mm to (60.5, 44.1), turned to 180 degrees
- moved C6 216.3 mm to (54.6, 34.8)
- moved C9 215.1 mm to (58.0, 37.1), turned to 90 degrees
- moved LED3 211.3 mm to (45.7, 43.6), turned to 270 degrees
- moved MOTOR1 204.7 mm to (52.1, 41.4), turned to 180 degrees
- moved R5 192.7 mm to (41.0, 28.4), turned to 270 degrees
- moved U$6 167.5 mm to (33.5, 21.0), turned to 180 degrees
- moved C7 47.4 mm to (60.5, 6.35), turned to 90 degrees
- moved C8 40.3 mm to (56.0, 6.99), turned to 90 degrees
- moved R9 31.6 mm to (43.6, 15.0), turned to 180 degrees
- moved MOTOR0 31.1 mm to (49.9, 10.7), turned to 180 degrees
- moved OUT_MOT0 30.5 mm to (59.4, 13.3)
- moved C5 29.2 mm to (42.0, 8.38), turned to 180 degrees
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Connections:
- removed net N$10: U$1.GND@3, U$5.GND@3
- removed net N$11: U$1.SCK, U$5.SCK
- removed net N$13: U$1.RESET_ICSP, U$5.RESET_ICSP
- removed net N$3: U$1.MISO, U$5.MISO
- removed net N$34: U$1.GND, U$5.GND
- removed net N$38: C12.1, MOTOR2.1
- removed net N$40: C12.2, MOTOR2.2
- removed net N$41: C13.1, MOTOR2.3
- removed net N$42: LED4.C, MOTOR2.18
- removed net N$43: LED4.A, R6.2
- removed net N$46: MOTOR2.10, MOTOR2.5, OUT_MOT2.1
- removed net N$47: MOTOR2.7, MOTOR2.8, OUT_MOT2.2
- removed net N$48: C16.1, MOTOR3.1
- removed net N$49: C16.2, MOTOR3.2
- removed net N$5: U$1.5V, U$5.5V
- removed net N$50: C17.1, MOTOR3.3
- removed net N$51: LED5.C, MOTOR3.18
- removed net N$52: LED5.A, R8.2
- removed net N$53: MOTOR3.10, MOTOR3.5, OUT_MOT3.1
- removed net N$54: MOTOR3.7, MOTOR3.8, OUT_MOT3.2
- removed net N$8: U$1.MOSI, U$5.MOSI
- removed net V3POUT2: C15.1, MOTOR2.12, MOTOR2.13, MOTOR2.15
- removed net V3POUT3: C18.1, MOTOR3.12, MOTOR3.13, MOTOR3.15
- new net GND1: U1.GND1
- new net GND2: U1.GND2
- net +12V: now also ALIM_V+.1; no longer C13.2, C17.2, MOTOR2.11, MOTOR2.4, MOTOR3.11, MOTOR3.4, PWR.1
- net /RST: now also U1.RESET; no longer U$1.RESET, U$5.RESET
- net A0: no longer TP5.P$1
- net A1: no longer TP4.P$1
- net ADC2: no longer MOTOR2.6, MOTOR2.9, R7.1
- net ADC3: no longer MOTOR3.6, MOTOR3.9, R15.1
- net GND: now also ALIM_GND.1; no longer C15.2, C18.2, MOTOR2.14, MOTOR2.28, MOTOR2.29, MOTOR3.14, MOTOR3.28, MOTOR3.29, PWM_ACCES.2, PWM_ACCES1.2, PWR1.1, R15.2, R7.2
- net GND_CLEAN: now also ALIM_GND.2, U1.GND; no longer PWR1.2, U$1.GND@1, U$1.GND@2, U$5.GND@1, U$5.GND@2
- net N$1: now also U1.IOREF; no longer U$1.IOREF, U$5.IOREF
- net N$15: now also U1.A5; no longer U$1.A5, U$5.A5
- net N$17: now also U1.A4; no longer U$1.A4, U$5.A4
- net N$2: now also U1.RESERVED; no longer U$1.RESERVED, U$5.RESERVED
- net N$20: now also U1.A0; no longer U$1.A0, U$5.A0
- net N$21: now also U1.A1; no longer U$1.A1, U$5.A1
- net N$22: now also U1.A2; no longer U$1.A2, U$5.A2
- net N$23: now also U1.A3; no longer U$1.A3, U$5.A3
- net N$24: now also U1.D0; no longer U$1.D0, U$5.D0
- net N$25: now also U1.D1; no longer U$1.D1, U$5.D1
- net N$26: now also U1.D2; no longer U$1.D2, U$5.D2
- net N$27: now also U1.D4; no longer U$1.D4, U$5.D4
- net N$28: now also U1.D7; no longer U$1.D7, U$5.D7
- net N$29: now also U1.D8; no longer U$1.D8, U$5.D8
- net N$30: now also U1.D12; no longer U$1.D12, U$5.D12
- net N$31: now also U1.D13; no longer U$1.D13, U$5.D13
- net N$32: now also U1.AREF; no longer U$1.AREF, U$5.AREF
- net N$4: now also U1.D9; no longer U$1.D9, U$5.D9
- net N$9: now also U1.5V; no longer U$1.5V_ICSP, U$5.5V_ICSP
- net PWM0: no longer PWM_ACCES.4
- net PWM0A: now also U1.D6; no longer U$1.D6, U$5.D6
- net PWM0B: now also U1.D5; no longer U$1.D5, U$5.D5
- net PWM1: no longer PWM_ACCES.3
- net PWM1B: now also U1.D10; no longer U$1.D10, U$5.D10
- net PWM2: no longer PWM_ACCES.6
- net PWM2A: now also U1.D11; no longer U$1.D11, U$5.D11
- net PWM2B: now also U1.D3; no longer U$1.D3, U$5.D3
- net PWM3: no longer PWM_ACCES.5
- net PWM4: no longer MOTOR2.21, PWM_ACCES1.4
- net PWM5: no longer MOTOR2.20, PWM_ACCES1.3
- net PWM6: no longer MOTOR3.21, PWM_ACCES1.6
- net PWM7: no longer MOTOR3.20, PWM_ACCES1.5
- net SCL_CLEAN: now also U1.SCL; no longer U$1.SCL, U$5.SCL
- net SDA_CLEAN: now also U1.SDA; no longer U$1.SDA, U$5.SDA
- net VCC: no longer MOTOR2.16, MOTOR2.17, MOTOR2.19, MOTOR2.23, MOTOR2.24, MOTOR2.25, MOTOR2.26, MOTOR2.27, MOTOR3.16, MOTOR3.17, MOTOR3.19, MOTOR3.23, MOTOR3.24, MOTOR3.25, MOTOR3.26, MOTOR3.27, PWM_ACCES.1, PWM_ACCES1.1, R6.1, R8.1
- net VCC_CLEAN: now also U1.3V; no longer U$1.3V, U$5.3V
- net VIN_ARDUINO: now also ALIM_V+.2, U1.VIN; no longer PWR.2, U$1.VIN, U$5.VIN
Routing:
- net VCC_CLEAN: track 0.00 -> 98.0 mm
- net VIN_ARDUINO: track 0.00 -> 30.7 mm
- net N$16: track 0.00 -> 26.0 mm
- net N$33: track 0.00 -> 22.9 mm
- net A1: track 17.1 -> 0.00 mm, vias 1 -> 0
- net A0: track 13.4 -> 0.00 mm, vias 1 -> 0
- net VCC: track 3.81 -> 16.8 mm
- net N$140: track 0.00 -> 11.5 mm
- net N$7: track 0.00 -> 7.47 mm
- net N$35: track 0.00 -> 6.36 mm
- net +12V: track 22.0 -> 16.3 mm
- net SCL: track 0.00 -> 3.76 mm
- net SDA: track 0.27 -> 3.97 mm
- net PWM0B: track 3.48 -> 0.00 mm
- net N$133: track 6.02 -> 2.83 mm
Other:
- board size 68.6 x 53.3 mm -> 65.8 x 53.5 mm
- board text added: "3V3LDO"
- board text added: "A0"
- board text added: "A1"
- board text added: "ALIM_GND"
- board text added: "ALIM_V+"
- board text added: "C1"
- board text added: "C10"
- board text added: "C11"
- board text added: "C14"
- board text added: "C2"
- board text added: "C3"
- board text added: "C4"
- board text added: "C5"
- board text added: "C6"
- board text added: "C7"
- board text added: "C8"
- board text added: "C9"
- board text added: "IC1"
- board text added: "IN_MOT1"
- board text added: "LED2"
- board text added: "LED3"
- board text added: "MOTOR0"
- board text added: "OUT_MOT0"
- board text added: "OUT_MOT1"
- board text added: "Q1"
- board text added: "R1"
- board text added: "R10"
- board text added: "R11"
- board text added: "R12"
- board text added: "R13"
- board text added: "R14"
- board text added: "R2"
- board text added: "R3"
- board text added: "R5"
- board text added: "R9"
- board text removed: "(3A max)"
- board text removed: "1.2A per motor"
- board text removed: "2 steppers"
- board text removed: "3v"
- board text removed: "4 DC motors"
- board text removed: "GND"
- board text removed: "Jumper"
- board text removed: "M2"
- board text removed: "M3"
- board text removed: "M4"
- board text removed: "Servo 1"
- board text removed: "VIN"
- board text removed: "logic:"
