File: hard/balise_infrarouge/cartev0/recepteur/recepteur_led.brd (EAGLE design)
At the start: 80 x 80 mm, 91 parts, among them IC3 4051D, IC4 4051D

Commit message: maj routage
Routing:
- net N$1: track 0.00 -> 3.02 mm
- net N$5: track 0.00 -> 2.02 mm
- net N$8: track 0.00 -> 1.64 mm
- net MUX0_C: track 12.5 -> 11.9 mm
- net GND: track 289.8 -> 290.3 mm
Other:
- board text added: "Bottom"
