File: hard/carteProto/carteProtoV2.brd (EAGLE design)
At the start: 138.4 x 113 mm, 45 parts

Commit message: Avancement de a carte v2 e proto
Parts:
- added H1, H2, H3, H4: (no value), holes:3,2-PAD
- added SK1: (no value), jt-con-micromatch:AMP-215079-8
- added U$5: MMATCH-4-, jt-con-micromatch:AMP-215079-4
- renumbered BOUTON to BOUTONS
Connections:
- net N$24 renamed +9V
- removed net SERIAL2: JP1.3, JP5.3, R5.1, U$1.P$49
- new net SERIAL1: JP1.3, JP5.3, R5.1, U$1.P$10, U$1.P$49
- net +5V: now also SK1.1, U$5.1
- net DIR1: now also SK1.4
- net DIR2: now also SK1.6
- net DIR3: now also SK1.8
- net GNDA: now also H1.B3,2, H2.B3,2, H3.B3,2, H4.B3,2, SK1.2, U$5.2
- net N$6: now also U$5.4
- net N$8: now also U$5.3
- net PWM1: now also SK1.3
- net PWM2: now also SK1.5
- net PWM3: now also SK1.7
Routing:
- removed copper zone on layer 1, net GNDA
- removed copper zone on layer 16, net GNDA

Commit message: Carte proto V2
Fin des modification et du routage. Prête à être imprimée
Parts:
- added AUTRES: MMATCH-6-, jt-con-micromatch:AMP-215079-6
- added IN_5-9-12: (no value), con-weidmueller-sl35:90G-4
- added R10, R8, R9: 10k, SparkFun-Passives:0805
- SV2: device con-lstb:MA03-1 -> con-lsta:FE05-1
- moved C11 80.0 mm to (112.4, 3.81)
- moved IN_12V 70.9 mm to (126.4, 27.9), turned to 180 degrees
- moved LED_12V 69.5 mm to (115.6, 26.0), turned to 90 degrees
- moved R7 68.6 mm to (120.0, 26.0), turned to 180 degrees
- moved C9 63.7 mm to (121.9, 11.4)
- moved U$5 63.4 mm to (43.8, 27.3), turned to 270 degrees
- moved LED_5V 45.9 mm to (115.6, 45.1), turned to 90 degrees
- moved R6 44.5 mm to (120.0, 45.1), turned to 180 degrees
- moved JP1 44.4 mm to (123.8, 88.3)
- moved JP5 43.9 mm to (111.1, 88.3)
- moved R5 41.3 mm to (120.0, 89.5), turned to 270 degrees
- moved SK1 32.0 mm to (76.2, 26.7)
- moved IN_5V 28.2 mm to (126.4, 47.0)
- moved LED_TEMOIN1 24.8 mm to (129.5, 62.9)
- moved LED_TEMOIN2 24.8 mm to (129.5, 60.3)
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Connections:
- new net N$24: AUTRES.3, U$1.P$2
- new net N$26: AUTRES.5, U$1.P$1
- new net N$27: AUTRES.4, U$1.P$21
- new net N$28: AUTRES.6, U$1.P$20
- net +12V: now also IN_5-9-12.4
- net +5V: now also AUTRES.1, IN_5-9-12.2, SV2.1
- net +9V: now also IN_5-9-12.3
- net GNDA: now also AUTRES.2, IN_5-9-12.1, R10.1, R8.1, R9.1, SV2.5
- net N$21: now also SV2.4; no longer SV2.3
- net N$22: now also SV2.3; no longer SV2.2
- net N$23: now also SV2.2; no longer SV2.1
- net PWM1: now also R8.2
- net PWM2: now also R9.2
- net PWM3: now also R10.2
Routing:
- net +5V: track 0.00 -> 540.5 mm, vias 0 -> 8
- net SERIAL1: track 0.00 -> 199.0 mm, vias 0 -> 3
- net +12V: track 0.00 -> 134.2 mm, vias 0 -> 5
- net PWM3: track 0.00 -> 113.2 mm, vias 0 -> 2
- net +9V: track 0.00 -> 110.9 mm, vias 0 -> 1
- net PWM1: track 0.00 -> 79.4 mm, vias 0 -> 2
- net PWM2: track 0.00 -> 73.4 mm, vias 0 -> 2
- net DIR1: track 0.00 -> 72.6 mm, vias 0 -> 2
- net N$14: track 0.00 -> 68.5 mm, vias 0 -> 1
- net N$13: track 0.00 -> 65.4 mm, vias 0 -> 1
- net DIR2: track 0.00 -> 64.0 mm
- net N$12: track 0.00 -> 61.6 mm, vias 0 -> 1
- net DIR3: track 0.00 -> 56.7 mm, vias 0 -> 2
- net SHARP0: track 0.00 -> 51.1 mm
- net CHA_3: track 0.00 -> 47.8 mm
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- added copper zone on layer 1, net GNDA
- added copper zone on layer 16, net GNDA
Other:
- board size 138.4 x 113 mm -> 138.4 x 114.3 mm
- board text added: "Protocarte V2"
- board text removed: "Bluetooth"
- board text removed: "LED1"
- board text removed: "LED2"
- board text removed: "LED3"
- board text removed: "Protocarte V1"
