File: hard/carteProto/carteProtoV2.sch (EAGLE design)
At the start: 45 parts

Commit message: Avancement de a carte v2 e proto
Parts:
- removed BOUTON: MMATCH-6-, jt-con-micromatch:MMATCH-6-
- added BOUTONS: MMATCH-6-, jt-con-micromatch:MMATCH-6-
- added H1, H2, H3, H4: MOUNT-PAD-ROUND3.2, holes:MOUNT-PAD-ROUND3.2
- added SK1: (no value), jt-con-micromatch:MMATCH-8-PTH
- added U$5: MMATCH-4-, jt-con-micromatch:MMATCH-4-
Connections:
- net N$24 renamed +9V
- removed net SERIAL2: JP1.3, JP5.3, R5.1, U$1.PA_9/D8/PWM1-2/SERIAL1_TX
- new net SERIAL1: JP1.3, JP5.3, R5.1, U$1.GND/SERIAL1_RX, U$1.PA_9/D8/PWM1-2/SERIAL1_TX
- net +5V: now also BOUTONS.3, SK1.1, U$5.5; no longer BOUTON.3
- net DIR1: now also SK1.4
- net DIR2: now also SK1.6
- net DIR3: now also SK1.8
- net GNDA: now also BOUTONS.4, H1.MOUNT, H2.MOUNT, H3.MOUNT, H4.MOUNT, SK1.2, U$5.6; no longer BOUTON.4
- net N$17: now also BOUTONS.5; no longer BOUTON.5
- net N$18: now also BOUTONS.7; no longer BOUTON.7
- net N$19: now also BOUTONS.8; no longer BOUTON.8
- net N$20: now also BOUTONS.6; no longer BOUTON.6
- net N$6: now also U$5.8
- net N$8: now also U$5.7
- net PWM1: now also SK1.3
- net PWM2: now also SK1.5
- net PWM3: now also SK1.7
Other:
- note added: "Alimentation"
- moved on the sheet: C1, C11, C2, C3, C4, C5, C6, C7, C9, IN_12V, IN_5V, IN_9V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

Commit message: Carte proto V2
Fin des modification et du routage. Prête à être imprimée
Parts:
- added AUTRES: MMATCH-6-, jt-con-micromatch:MMATCH-6-
- added IN_5-9-12: (no value), con-weidmueller-sl35:90G-4
- added R10, R8, R9: 10k, SparkFun-Passives:RESISTOR0805-RES
- SV2: device con-lstb:MA03-1 -> con-lsta:FE05-1
Connections:
- new net N$24: AUTRES.5, U$1.PC_12/SPI3_MOSI
- new net N$26: AUTRES.7, U$1.PC_10/SPI3_SCK
- new net N$27: AUTRES.6, U$1.PD_2
- new net N$28: AUTRES.8, U$1.PC_11/SPI3_MISO
- net +12V: now also IN_5-9-12.4
- net +5V: now also AUTRES.3, IN_5-9-12.2, SV2.1
- net +9V: now also IN_5-9-12.3
- net GNDA: now also AUTRES.4, IN_5-9-12.1, R10.1, R8.1, R9.1, SV2.5
- net N$21: now also SV2.4; no longer SV2.3
- net N$22: now also SV2.3; no longer SV2.2
- net N$23: now also SV2.2; no longer SV2.1
- net PWM1: now also R8.2
- net PWM2: now also R9.2
- net PWM3: now also R10.2
