File: hard/carteBoutons/carteBoutonsV1.brd (EAGLE design)
At the start: 67.3 x 52.7 mm, 26 parts

Commit message: maj boutons
Connections:
- net GND: no longer H1.B3,2, H2.B3,2, H3.B3,2, H4.B3,2
Routing:
- net GND: vias 6 -> 7
Changed lines of the file:
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@@
 <layer number="16" name="Bottom" color="1" fill="1" visible="yes" active="yes"/>
 <layer number="17" name="Pads" color="2" fill="1" visible="yes" active="yes"/>
-<layer number="18" name="Vias" color="2" fill="1" visible="yes" active="yes"/>
+<layer number="18" name="Vias" color="14" fill="1" visible="yes" active="yes"/>
 <layer number="19" name="Unrouted" color="6" fill="1" visible="yes" active="yes"/>
 <layer number="20" name="Dimension" color="15" fill="1" visible="yes" active="yes"/>
@@
 <vertex x="-9.525" y="-10.16"/>
 </polygon>
-<contactref element="H4" pad="B3,2"/>
-<contactref element="H3" pad="B3,2"/>
-<contactref element="H2" pad="B3,2"/>
-<contactref element="H1" pad="B3,2"/>
 <contactref element="BT_12V" pad="1"/>
 <contactref element="BT_9V" pad="1"/>
@@
 <via x="-1.905" y="10.795" extent="1-16" drill="1.1"/>
 <via x="8.89" y="16.51" extent="1-16" drill="1.1"/>
-<via x="29.845" y="19.685" extent="1-16" drill="1.1"/>
+<via x="29.5275" y="17.4625" extent="1-16" drill="1.1"/>
 <via x="29.21" y="24.765" extent="1-16" drill="1.1"/>
 <via x="23.495" y="4.445" extent="1-16" drill="1.1"/>
+<via x="8.89" y="39.37" extent="1-16" drill="1.1"/>
 </signal>
 <signal name="N$15">
